Commit message: Wheel geometry: 440 mm wheel base, 512 mm-wide footprint, wheels in the model
Drive wheels are 192 mm diameter and 72 mm wide, mounted outside the 360 mm case with
368 mm between their inner faces: 440 mm centre to centre, 512 mm across the outsides.

- esp32_serial_bridge: wheel_base_m 0.22 -> 0.44 (turn commands were coming out at
  half the requested rate)
- nav2_params: footprint 495 x 512 mm, inflation 0.45 m local / 0.50 m global (corner
  radius 0.356 m), collision stop/slowdown zones 56 / 64 cm wide
- urdf: both wheels drawn to scale beside the case

Tested: Nav2 publishes the 495 x 512 mm footprint (+1 cm padding) and the new zones;
model shows both wheels; 18 unit tests pass.

File: src/securebot_ros/urdf/securebot.urdf (robot description, URDF)
Before this commit: robot securebot, 1 links, 0 joints
Links:
- added link left_wheel; visual cylinder length=0.072 radius=0.096
- added link right_wheel; visual cylinder length=0.072 radius=0.096
Joints:
- added joint left_wheel_joint: type fixed, parent base_link, child left_wheel, origin xyz=0 0.22 0 rpy=0 0 0
- added joint right_wheel_joint: type fixed, parent base_link, child right_wheel, origin xyz=0 -0.22 0 rpy=0 0 0
